File: trackpals/trackpals.kicad_sch (KiCad schematic)
At the start: 91 parts, among them J1 Battery Connector, J2 CONUFL001-SMD-T, J3 CONUFL001-SMD-T, J6 Conn_01x02_Socket, Q1 BSS138, Q2 BSS138, Q3 AO4459, Q4 BC848, SW1 SW_Push, SW2 SW_Push, SW4 SW_Push, SW5 SW_Push, U1 BQ24040DSQR, U2 CH340C, U3 TPL5110, U4 ESP32-WROOM-32, U5 TPS73733DCQR

Commit message: -
Parts:
- removed BT1: Battery_Cell, symbol Device:Battery_Cell
- added BAT1: ~, ProLib_pcs_2026-02-08:BAT-SMD_CR1202, symbol Symbols_track:3000
- added C16: 100uF, Capacitor_SMD:C_1210_3225Metric_Pad1.33x2.70mm_HandSolder, symbol Device:C_Polarized
- added C18, C20, C22: 22pF, Capacitor_SMD:C_0603_1608Metric_Pad1.08x0.95mm_HandSolder, symbol Device:C
- added C19, C23, C24, C31: 100nF, Capacitor_SMD:C_0603_1608Metric_Pad1.08x0.95mm_HandSolder, symbol Device:C
- added C21: 1uF, Capacitor_SMD:C_0805_2012Metric_Pad1.18x1.45mm_HandSolder, symbol Device:C
- added C27: 4.7uF, Capacitor_Tantalum_SMD:CP_EIA-3528-12_Kemet-T_HandSolder, symbol Device:C_Polarized
- added C29: 330uF, Capacitor_Tantalum_SMD:CP_EIA-7343-31_Kemet-D_HandSolder, symbol Device:C_Polarized
- added Card2: DS1138-02-06SS4BOR, SolX:SIM-SMD_DS1138-02-06SS4BOR, symbol easyeda2kicad:DS1138-02-06SS4BOR
- added D10: ESDA6V1-5SC6, Package_TO_SOT_SMD:SOT-23-6, symbol Power_Protection:ESDA6V1-5SC6
- added D12, D13: LED, LED_SMD:LED_0805_2012Metric_Pad1.15x1.40mm_HandSolder, symbol Device:LED
- added J5: Conn_01x03_Socket, Jumper:SolderJumper-3_P1.3mm_Open_Pad1.0x1.5mm, symbol Connector:Conn_01x03_Socket
- added J6: CONUFL001-SMD-T, SolX:IPEX-SMD_3P-L2.6-W2.6-LS3.0, symbol ICPH:CONUFL001-SMD-T
- added JP12, JP7: SolderJumper_2_Open, Jumper:SolderJumper-2_P1.3mm_Open_Pad1.0x1.5mm, symbol Jumper:SolderJumper_2_Open
- added Q5: BC848, Package_TO_SOT_SMD:SOT-23, symbol Transistor_BJT:BC848
- added R19, R34, R35: 1K, Resistor_SMD:R_0603_1608Metric_Pad0.98x0.95mm_HandSolder, symbol Device:R
- added R23: 4.7K, Resistor_SMD:R_0603_1608Metric_Pad0.98x0.95mm_HandSolder, symbol Device:R
- added R24: 47K, Resistor_SMD:R_0805_2012Metric_Pad1.20x1.40mm_HandSolder, symbol Device:R
- added R25, R26, R27: 53, Resistor_SMD:R_0805_2012Metric_Pad1.20x1.40mm_HandSolder, symbol Device:R
- added R28, R30: 43K, Resistor_SMD:R_0805_2012Metric_Pad1.20x1.40mm_HandSolder, symbol Device:R
- added R29: 100K, Resistor_SMD:R_0805_2012Metric_Pad1.20x1.40mm_HandSolder, symbol Device:R
- added R31: 470, Resistor_SMD:R_0805_2012Metric_Pad1.20x1.40mm_HandSolder, symbol Device:R
- added U11: SIM800C, RF_GSM:SIMCom_SIM800C, symbol RF_GSM:SIM800C
- added U6: TXS0102DCT, Package_SO:SSOP-8_2.95x2.8mm_P0.65mm, symbol Logic_LevelTranslator:TXS0102DCT
- added U7: MIC29302WU, Package_TO_SOT_SMD:TO-263-5_TabPin3, symbol Regulator_Linear:MIC29302WU
- D1: renamed from D9; footprint (none) -> Diode_SMD:D_0805_2012Metric
- L1: footprint (none) -> Inductor_SMD:L_0603_1608Metric_Pad1.05x0.95mm_HandSolder
- Q1: renamed from Q3; footprint powergate:SOP-8_L5.0-W4.0-P1.27-LS6.2-BL -> Footprint_track:SOP-8_L5.0-W4.0-P1.27-LS6.2-BL
- U1: footprint tanimoji:WSON-10_L2.0-W2.0-P0.40-BL-EP -> Footprint_track:WSON-10_L2.0-W2.0-P0.40-BL-EP
- U10: renamed from U8; value ~ -> HK24C32HA-USR-B; footprint (none) -> Footprint_track:SOP-8_L5.0-W4.0-P1.27-LS6.2-BL
- U2: renamed from U5; footprint tanimoji:SOT-223-6_L6.5-W3.5-P1.27-BL -> Footprint_track:SOT-223-6_L6.5-W3.5-P1.27-BL
- U9: renamed from U7; value ~ -> NEO-6M-GPS; footprint (none) -> Footprint_track:XCVR_NEO-6M-GPS
- USB1: footprint tanimoji:USB-C-SMD_TYPE-C16PIN -> Footprint_track:USB-C-SMD_TYPE-C16PIN
- renumbered C18 to C1, C11 to C10, C12 to C11, C13 to C12, C14 to C13, C4 to C14, C5 to C15, C6 to C17, C1 to C2, C7 to C25, C8 to C26, C22 to C28, C19 to C3, C21 to C30, C17 to C32, C20 to C33, C16 to C4, C15 to C5, C9 to C6, C10 to C7, C2 to C8, C3 to C9, D5 to D11, D11 to D14, D1 to D2, D2 to D3, D6 to D4, D7 to D5, D3 to D6, D4 to D7, D10 to D9, J3 to J1, J6 to J2, J1 to J3, J2 to J4, JP9 to JP11, JP5 to JP3, JP6 to JP4, JP3 to JP5, JP4 to JP6, JP7 to JP8, JP8 to JP9, Q1 to Q2, Q2 to Q3, R3 to R1, R7 to R10, R14 to R11, R15 to R12, R8 to R13, R9 to R14, R10 to R15, R18 to R16, R16 to R17, R17 to R18, R21 to R2, R13 to R20, R11 to R21, R23 to R22, R4 to R3, R12 to R32, R22 to R33, R24 to R36, R1 to R4, R2 to R5, R5 to R6, R19 to R7, R6 to R8, R20 to R9, SW4 to SW1, SW5 to SW2, SW1 to SW3, SW2 to SW4, U2 to U4, U6 to U5, U4 to U8
Connections:
- net +3.3V: now also C19.2, R19.1, U6.3 (VCCA)
- net GND: now also BAT1.3 (-), C16.2, C18.1, C19.1, C20.1, C21.2, C22.1, C23.1, C24.1, C27.2, C29.2, C31.2, Card2.C4 (GND), D10.2 (GND), J5.1 (Pin_1), J6.2, J6.3, Q5.2 (E), R24.2, R28.2, R30.2, R31.2, R34.2, R35.2, U11.13 (GND), U11.19 (GND), U11.21 (GND), U11.27 (GND), U11.30 (GND), U11.31 (GND), U11.33 (GND), U11.36 (GND), U11.37 (GND), U11.8 (GND), U6.2 (GND), U7.3 (GND)
- net GPS_RX: now also U8.28 (IO17); no longer U8.12 (IO27)
- net GPS_TX: now also U8.27 (IO16); no longer U8.13 (IO14)
- net GSM_PWRKEY: now also JP7.1 (A), R23.1; no longer U8.26 (IO4)
- net SIM_CARD_CLK: now also Card2.C3 (CLK), D10.4 (IO3), R26.2
- net SIM_CARD_IO: now also Card2.C6 (IO), D10.6 (IO5), R27.2
- net SIM_CARD_RST: now also Card2.C2 (RST), D10.3 (IO2), R25.2
- net SIM_CARD_VCC: now also C24.2, Card2.C1 (VCC), D10.1 (IO1), U11.18 (SIM_VDD)
- net SIM_RESET: now also JP12.1 (A); no longer C32.2, R33.2, U8.11 (IO26)
- net VDC: now also C16.1, C21.1, J5.3 (Pin_3), U7.2 (VIN)
- net at R36.2, U9.22 (V_BACKUP): now also BAT1.1 (+), BAT1.2 (+)
- net GSM_TX: now reaches U8.16 (IO13)
- net GSM_TX: now also U5.32 (UART_TXD), U6.5 (A1)
- net ESP_RX2 renamed GSM_RX
- net GSM_RX: now also U8.13 (IO14), U6.4 (A2); no longer U8.28 (IO17)
- removed net ESP_TX2: U5.32 (UART_TXD), U8.27 (IO16)
- new net: J5.2 (Pin_2), U7.1 (EN)
- new net: R28.1, R29.2, R30.1, U7.5 (ADJ)
- new net: D12.1 (K), R34.1
- new net: D12.2 (A), U11.42 (STATUS)
- new net: D13.1 (K), R35.1
- new net: D13.2 (A), U11.41 (NETLIGHT)
- new net: C32.2, JP12.2 (B), R33.2, U8.11 (IO26)
- new net: R19.2, U6.6 (OE)
- new net: Q5.1 (B), R23.2, R24.1
- new net: Q5.3 (C), U11.39 (~{PWRKEY})
- new net: C27.1, U11.28 (VRTC)
- new net: U11.1 (UART1_TXD), U6.8 (B1)
- new net: U11.2 (UART1_RXD), U6.1 (B2)
- new net: J6.1, U11.32 (GSM_ANT)
- new net: JP7.2 (B), U8.26 (IO4)
- new net GSM_VCC: C29.1, C31.1, R29.1, R31.1, U11.34 (VBAT), U11.35 (VBAT), U7.4 (VOUT)
- new net GSM_VDD_2V8: C23.2, U11.40 (VDD_EXT), U6.7 (VCCB)
- new net SIM_CLK: C20.2, R26.1, U11.16 (SIM_CLK)
- new net SIM_DAT: C18.2, R27.1, U11.15 (SIM_DATA)
- new net SIM_RST: C22.2, R25.1, U11.17 (SIM_RST)
- no-connect marks 71 -> 106
Other:
- note added: "GSM"
