File: trackpals/trackpals.kicad_pcb (KiCad board)
At the start: 2 copper layers, 70 x 50 mm, 100 parts, among them J1 CONUFL001-SMD-T, J2 Conn_01x02_Socket, J3 Battery Connector, J4 CONUFL001-SMD-T, Q1 BC848, Q2 AO4459, Q3 BSS138, Q4 BSS138, SW1 SW_Push, SW2 SW_Push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

Commit message: - DONE PCB
Parts:
- added H2: MountingHole, MountingHole:MountingHole_3.2mm_M3_Pad_TopBottom, F.Cu at (160.3, 139.0)
- added H2: MountingHole, MountingHole:MountingHole_3.2mm_M3_Pad_TopBottom, F.Cu at (160.3, 96.1)
- added H2: MountingHole, MountingHole:MountingHole_3.2mm_M3_Pad_TopBottom, F.Cu at (97.2, 96.1)
- added H2: MountingHole, MountingHole:MountingHole_3.2mm_M3_Pad_TopBottom, F.Cu at (97.2, 139.0)
- moved JP8 8.94 mm to (109.9, 113.0), turned to 90 degrees
- moved JP7 8.94 mm to (107.3, 113.0), turned to 90 degrees
- moved J3 6.19 mm to (159.7, 105.1)
- moved C8 5.45 mm to (154.7, 137.2), turned to 0 degrees
- moved C7 3.91 mm to (154.7, 135.1), turned to 0 degrees
- moved SW2 2.97 mm to (103.7, 132.2)
- moved C21 2.97 mm to (102.0, 135.6)
- moved R25 2.97 mm to (106.0, 135.6)
- moved C5 2.96 mm to (112.3, 139.6)
- moved R10 2.96 mm to (112.4, 135.8)
- moved C13 2.39 mm to (151.6, 127.9)
- moved JP3 2.39 mm to (150.8, 128.7)
- moved U4 2.39 mm to (154.8, 132.3)
- moved R13 2.39 mm to (150.7, 130.7)
- moved R15 2.39 mm to (149.5, 127.9)
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Routing:
- net +3.3V: track 0.00 -> 194.5 mm, vias 0 -> 8
- net SIM_CARD_GND: track 2.24 -> 117.4 mm, vias 2 -> 72
- net VBAT: track 0.00 -> 105.4 mm, vias 0 -> 8
- net VDC: track 0.00 -> 99.1 mm, vias 0 -> 7
- net ESP_TX: track 0.00 -> 74.8 mm, vias 0 -> 2
- net ESP_RX: track 0.00 -> 69.2 mm, vias 0 -> 2
- net ESP_EN: track 0.00 -> 65.8 mm, vias 0 -> 2
- net TIMER_DONE: track 0.00 -> 54.8 mm, vias 0 -> 2
- net ESP_I0: track 0.00 -> 46.7 mm, vias 0 -> 2
- net +5V: track 0.00 -> 45.0 mm, vias 0 -> 5
- net Net-(U8-V_BACKUP): track 0.00 -> 42.4 mm, vias 0 -> 4
- net SIM_CARD_VCC: track 0.00 -> 39.0 mm, vias 0 -> 3
- net SCL2: track 0.00 -> 36.8 mm, vias 0 -> 1
- net SIM_CARD_CLK: track 0.00 -> 36.6 mm, vias 0 -> 1
- net SIM_CARD_RST: track 0.00 -> 36.0 mm, vias 0 -> 1
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- added copper zone on B.Cu, net SIM_CARD_GND
- added copper zone on F.Cu, net SIM_CARD_GND
- added copper zone on In1.Cu, net SIM_CARD_GND
- added copper zone on In2.Cu, net SIM_CARD_GND
Other:
- outline, holes or cut-outs redrawn
- copper layers 2 -> 4
- board text added: "+"
- board text added: "-"

Commit message: updated tssop
Parts:
- U9: footprint Footprint_track:SOP-8_L5.0-W4.0-P1.27-LS6.2-BL -> Package_SO:TSSOP-8_4.4x3mm_P0.65mm
- moved JP5 0.90 mm to (154.5, 105.6)
- moved U9 0.63 mm to (110.6, 100.6), turned to 0 degrees
- turned R21 to 90 degrees
Connections:
- R21 pad 1: SIM_CARD_GND -> Net-(U2-TS)
- R21 pad 2: Net-(U2-TS) -> SIM_CARD_GND
- U7 pad 11: Net-(JP11-B) -> unconnected-(U7-IO26-Pad11)
Routing:
- net SDA2: track 31.0 -> 32.4 mm
- net VDC: track 99.1 -> 98.3 mm
- net SCL2: track 36.8 -> 37.5 mm
- net Net-(JP5-C): track 5.41 -> 6.11 mm
Other:
- board text added: "*"
- board text added: "3.3V LED"
- board text added: "DM_EN"
- board text added: "GND"
- board text added: "IO0"
- board text added: "ISET"
- board text added: "ISET2"
- board text added: "PWRKEY"
- board text added: "RST"
- board text added: "RX"
- board text added: "SCL"
- board text added: "SDA"
- board text added: "TMR_DONE"
- board text added: "TX"
- board text added: "VBAT_IN"
- board text added: "VDC"
- board text added: "VDC_LED"
